Commit message: Correct carma fixed xacro and launch files
Add start_gazebo

To test carma do
roslaunch manipulator_tether_lifting start_gazebo.launch gravity:=false

Let gazebo initialize properly

spawn_carma_fixed_w_controllers.launch

spawns the carma plus the joint controllers

base_carma_on_ceiling{0,1}.xacro provides the xacro for the robot

File: urdf/carma/base_carma.xacro (robot description, xacro)
@@ -31,9 +31,12 @@
   <xacro:property name="manipulator_position_z" value="-0.0" /> <!-- [m] -->
   <!-- chosen as a tenth of the friction... -->
-  <xacro:property name="damping" value="0.03" /> <!-- [(N*m)/(rad/s)] -->
+  <!-- <xacro:property name="damping" value="0.03" /> --> <!-- [(N*m)/(rad/s)] -->
+  <xacro:property name="damping" value="0.0" /> <!-- [(N*m)/(rad/s)] -->
   <!-- chosen as half of the torque the base joint requires to keep the arm horizontal... -->
-  <xacro:property name="friction" value="0.3" /> <!-- [N*m] -->
+  <!-- <xacro:property name="friction" value="0.3" /> --> <!-- [N*m] -->
+  <xacro:property name="friction" value="0.0" /> <!-- [N*m] -->
   <!-- effort: gearmotor torque = 5 kg*cm, bevel gear ratio is 1:2, so 1 N*m -->
-  <xacro:property name="effort" value="1" /> <!-- [N*m] -->
+  <!-- <xacro:property name="effort" value="1" /> --> <!-- [N*m] -->
+  <xacro:property name="effort" value="10" /> <!-- [N*m] -->
   <!-- Included URDF Files -->
   <xacro:include filename="$(find manipulator_tether_lifting)/urdf/carma/macro_carma.xacro"/>

File: urdf/carma/base_carma_on_ceiling1.xacro (robot description, xacro)
@@ -1,39 +1,23 @@
 <?xml version="1.0"?>
-<!-- -->
+<!--
+  carma with end-effector as root link, and attached to world (end-effector attached to world)
+-->
 <robot name="carma_on_ceiling" xmlns:xacro="http://ros.org/wiki/xacro">
   <xacro:property name="namespace" value="$(arg namespace)"/>
-  <!-- add carma -->
   <xacro:property name="carma_namespace" value="${namespace}/carma"/>
-  <xacro:include filename="$(find manipulator_tether_lifting)/urdf/carma/base_carma.xacro"/>
+  <xacro:include filename="$(find manipulator_tether_lifting)/urdf/carma/base_carma_reversed.xacro"/>
   <link name="world">
   </link>
-  <joint name="${namespace}/joint_ceiling_world" type="fixed">
-     <origin xyz="0 0 0" rpy="0 0 0"/>
+  <joint name="${namespace}/carma/joint1" type="fixed">
+      <origin xyz="0 0 0" rpy="0 0 0"/>
       <parent link="world"/>
-      <child link="${namespace}/link_ceiling"/>
-  </joint>
-  <link name="${namespace}/link_ceiling">
-   <inertial>
-     <origin xyz="0 0 0" rpy="0 0 0"/>
-     <mass value="1"/>
-     <inertia ixx="1" ixy="0" ixz="0"
-              iyy="1" iyz="0"
-              izz="1" />
-   </inertial>
-   <visual>
-     <origin xyz="0 0 0" rpy="0 0 0" />
-     <geometry>
-       <box size="0.5 0.5 0.1" />
-     </geometry>
-     <material name="Cyan">
-       <color rgba="0 1.0 1.0 1.0"/>
-     </material>
-   </visual>
-  </link>
-  <joint name="${namespace}/joint_ceiling_link1" type="continuous">
-      <origin xyz="0 0 0" rpy="0 0 0"/>
-      <axis xyz="0 1 0" />
-      <parent link="${namespace}/link_ceiling"/>
-      <child link="${namespace}/carma/link1"/>
+      <child link="${namespace}/carma/link5"/>
    </joint>
+  <gazebo>
+    <plugin name="gazebo_ros_control" filename="libgazebo_ros_control.so">
+      <!-- <robotNamespace>${namespace}</robotNamespace> -->
+      <!-- <robotParam>${namespace}/robot_description</robotParam> -->
+      <robotNamespace></robotNamespace>
+    </plugin>
+  </gazebo>
 </robot>

File: urdf/carma/base_carma_reversed.xacro (robot description, xacro)
@@ -10,12 +10,12 @@
   <xacro:property name="mass_end_effector" value="0.038" /> <!-- [kg] -->
   <!-- TODO: low values here screw up simulation -->
-  <!-- <xacro:property name="inertia_zz_link1" value="0.000253151228084876" />   -->
-  <!-- <xacro:property name="inertia_zz_link2" value="0.000108770447476707" />   -->
-  <!-- <xacro:property name="inertia_zz_link3" value="3.47458286569986e-05" />   -->
-  <!-- <xacro:property name="inertia_zz_link4" value="3.42053994711421e-05" />   -->
-  <xacro:property name="inertia_zz_link1" value="0.00253151228084876" /> <!-- [kg*m^2] -->
-  <xacro:property name="inertia_zz_link2" value="0.00108770447476707" /> <!-- [kg*m^2] -->
-  <xacro:property name="inertia_zz_link3" value="3.47458286569986e-03" /> <!-- [kg*m^2] -->
-  <xacro:property name="inertia_zz_link4" value="3.42053994711421e-03" /> <!-- [kg*m^2] -->
+  <xacro:property name="inertia_zz_link1" value="0.000253151228084876" />
+  <xacro:property name="inertia_zz_link2" value="0.000108770447476707" />
+  <xacro:property name="inertia_zz_link3" value="3.47458286569986e-05" />
+  <xacro:property name="inertia_zz_link4" value="3.42053994711421e-05" />
+  <!-- <xacro:property name="inertia_zz_link1" value="0.00253151228084876" />  -->
+  <!-- <xacro:property name="inertia_zz_link2" value="0.00108770447476707" />  -->
+  <!-- <xacro:property name="inertia_zz_link3" value="3.47458286569986e-03" /> -->
+  <!-- <xacro:property name="inertia_zz_link4" value="3.42053994711421e-03" /> -->
   <xacro:property name="length_x_link1" value="0.173000000000000" /> <!-- [m] -->
   <xacro:property name="length_x_link2" value="0.122000000000000" /> <!-- [m] -->
